Commit message: Add files via upload

File: testarm_urdf/urdf/testarm_urdf.urdf (robot description, URDF)
Before this commit: robot testarm_urdf, 4 links, 3 joints
Links:
- link l3: mass 339.624762377846 -> 339.62
Joints:
- joint j1: axis 0 0 0 -> 0 0 1; limit lower=0 upper=3.142 effort=300 velocity=3 -> lower=0 upper=3.1412 effort=300 velocity=3; origin xyz=0 0.1524 0.59921 rpy=1.5708 0 0 -> xyz=0.00011944 0 0.34027 rpy=0 0 0
- joint j2: axis 0 0 0 -> 0 -1 0; origin xyz=0 0.254 0.0508 rpy=0 0 0 -> xyz=-0.00011944 0 0.18012 rpy=0 0 0
- joint j3: axis 0 0 0 -> 0 -1 0; limit lower=-1.57 upper=1.57 effort=200 velocity=3 -> lower=0 upper=3.142 effort=300 velocity=3; origin xyz=-0.34822 0 -0.0508 rpy=0 0 1.5708 -> xyz=0 0 0.39751 rpy=0 0 0
